File: hw/baseline_project.kicad_sch (KiCad schematic)
At the start: 20 parts, among them J101 EXT_3V3, Q101 IRLD024PBF, SW101 UP, SW102 DOWN, SW103 LEFT, SW104 RIGHT, SW105 MODE, U101 EK-TM4C123GXL, U102 ESP8266-1, U103 Adafruit ST7735R

Commit message: Hardware
Parts:
- removed C101: 100nF, ECE445L:C_Axial_200mil, symbol ECE445L:C
- removed C103: 4.7uF, ECE445L:CP_Radial_Tantal200mil, symbol ECE445L:C_Polarized
- removed D101: 1V0, Diode_THT:D_5W_P12.70mm_Horizontal, symbol Device:D_Small
- removed H1, H2, H3, H4: ~, ECE445L:MountingHole_4_40, symbol ECE445L:MountingHole
- removed J101: EXT_3V3, Connector_Samtec_HPM_THT:Samtec_HPM-02-01-x-S_Straight_1x02_Pitch5.08mm, symbol Connector_Generic:Conn_01x02
- removed R101: 10k, ECE445L:R_Axial_DIN0204_L3.6mm_D1.6mm_P7.62mm_Horizontal, symbol ECE445L:R_0.125W
- removed SW104: RIGHT, Button_Switch_THT:SW_PUSH_6mm, symbol Switch:SW_Push
- removed SW105: MODE, Button_Switch_THT:SW_PUSH_6mm, symbol Switch:SW_Push
- removed U102: ESP8266-1, ECE445L:PinHeader_2x04_P2.54mm_Vertical, symbol ECE445L:ESP8266-1
- added C1: .1 microFarad, symbol Device:C_Polarized
- SW101: value UP -> DOWN
- SW103: value LEFT -> DOWN
Connections:
- net +3V3: now also C1.1
- net PB1: no longer R102.1
- net PB4: now also R102.1
- net PC4: no longer SW101.2
- net PC6: no longer SW103.2
- net PC7: no longer SW102.2
- net PE0: now also SW101.2
- net PE1: now also SW102.2
- net PE2: now also SW103.2
- net at LS101.2, Q101.1 (D), Q101.2 (D): now also C1.2
